File: hardware/adb.sch (EAGLE design)
At the start: 10 parts, among them U1 Tiny85-20-SMT

Commit message: hardware: AVR reset pulled high.
Parts:
- added R4: 10K, SparkFun-Passives:RESISTOR0805-RES
Connections:
- net RESET: now also R4.1
- net VCC: now also R4.2
Other:
- moved on the sheet: R1, R2
Changed lines of the file:
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@@
 <setting verticaltext="up"/>
 </settings>
-<grid distance="0.1" unitdist="inch" unit="inch" style="lines" multiple="1" display="yes" altdistance="0.01" altunitdist="inch" altunit="inch"/>
+<grid distance="0.1" unitdist="inch" unit="inch" style="lines" multiple="1" display="no" altdistance="0.01" altunitdist="inch" altunit="inch"/>
 <layers>
 <layer number="1" name="Top" color="4" fill="1" visible="no" active="no"/>
@@
 <part name="R3" library="SparkFun-Passives" deviceset="RESISTOR" device="0805-RES" value="2K2"/>
 <part name="SUPPLY4" library="SparkFun-Aesthetics" deviceset="VCC" device=""/>
+<part name="R4" library="SparkFun-Passives" deviceset="RESISTOR" device="0805-RES" value="10K"/>
+<part name="SUPPLY6" library="SparkFun-Aesthetics" deviceset="VCC" device=""/>
 </parts>
 <sheets>
@@
 <instance part="SUPPLY2" gate="G$1" x="88.9" y="50.8"/>
 <instance part="SUPPLY3" gate="G$1" x="27.94" y="17.78"/>
-<instance part="R2" gate="G$1" x="55.88" y="38.1"/>
-<instance part="R1" gate="G$1" x="48.26" y="43.18"/>
+<instance part="R2" gate="G$1" x="45.72" y="38.1"/>
+<instance part="R1" gate="G$1" x="53.34" y="43.18"/>
 <instance part="D1" gate="G$1" x="73.66" y="27.94" rot="R90"/>
 <instance part="D2" gate="G$1" x="78.74" y="22.86" rot="R90"/>
@@
 <instance part="R3" gate="G$1" x="73.66" y="48.26"/>
 <instance part="SUPPLY4" gate="G$1" x="78.74" y="50.8"/>
+<instance part="R4" gate="G$1" x="53.34" y="30.48"/>
+<instance part="SUPPLY6" gate="G$1" x="58.42" y="30.48"/>
 </instances>
 <busses>
@@
 <pinref part="SUPPLY4" gate="G$1" pin="VCC"/>
 <wire x1="78.74" y1="48.26" x2="78.74" y2="50.8" width="0.1524" layer="91"/>
+</segment>
+<segment>
+<pinref part="R4" gate="G$1" pin="2"/>
+<pinref part="SUPPLY6" gate="G$1" pin="VCC"/>
 </segment>
 </net>
@@
 <pinref part="U1" gate="G$1" pin="PB2(SCK/ADC1)"/>
 <pinref part="R2" gate="G$1" pin="1"/>
-<wire x1="30.48" y1="38.1" x2="50.8" y2="38.1" width="0.1524" layer="91"/>
+<wire x1="30.48" y1="38.1" x2="40.64" y2="38.1" width="0.1524" layer="91"/>
 </segment>
 <segment>
@@
 <wire x1="78.74" y1="38.1" x2="78.74" y2="25.4" width="0.1524" layer="91"/>
 <pinref part="R2" gate="G$1" pin="2"/>
-<wire x1="60.96" y1="38.1" x2="68.58" y2="38.1" width="0.1524" layer="91"/>
+<wire x1="50.8" y1="38.1" x2="68.58" y2="38.1" width="0.1524" layer="91"/>
 <junction x="78.74" y="38.1"/>
 <pinref part="USB1" gate="USB" pin="D-"/>
@@
 <segment>
 <pinref part="R1" gate="G$1" pin="2"/>
-<wire x1="53.34" y1="43.18" x2="73.66" y2="43.18" width="0.1524" layer="91"/>
+<wire x1="58.42" y1="43.18" x2="73.66" y2="43.18" width="0.1524" layer="91"/>
 <pinref part="D1" gate="G$1" pin="C"/>
 <wire x1="78.74" y1="43.18" x2="73.66" y2="43.18" width="0.1524" layer="91"/>
@@
 <pinref part="R1" gate="G$1" pin="1"/>
 <pinref part="U1" gate="G$1" pin="PB0(MOSI)"/>
-<wire x1="43.18" y1="43.18" x2="30.48" y2="43.18" width="0.1524" layer="91"/>
+<wire x1="48.26" y1="43.18" x2="30.48" y2="43.18" width="0.1524" layer="91"/>
 </segment>
 <segment>
@@
 <segment>
 <pinref part="U1" gate="G$1" pin="PB5(NRES)"/>
-<wire x1="30.48" y1="30.48" x2="38.1" y2="30.48" width="0.1524" layer="91"/>
-<label x="38.1" y="30.48" size="1.778" layer="95"/>
-</segment>
-<segment>
+<wire x1="30.48" y1="30.48" x2="48.26" y2="30.48" width="0.1524" layer="91"/>
+<pinref part="R4" gate="G$1" pin="1"/>
+</segment>
+<segment>

Commit message: hardware: polish; silk screen text etc.
Connections:
- net N$2 renamed PB4
- net N$5 renamed PB3
Changed lines of the file:
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@@
 <?xml version="1.0" encoding="utf-8"?>
 <!DOCTYPE eagle SYSTEM "eagle.dtd">
-<eagle version="7.1.0">
+<eagle version="7.2.0">
 <drawing>
 <settings>
@@
 </segment>
 </net>
-<net name="N$2" class="0">
+<net name="PB4" class="0">
 <segment>
 <pinref part="U1" gate="G$1" pin="PB4(ADC2)"/>
@@
 </segment>
 </net>
-<net name="N$5" class="0">
+<net name="PB3" class="0">
 <segment>
 <pinref part="U1" gate="G$1" pin="PB3(ADC3)"/>
